Commit message: temp

File: ros_ws/pmi_description/urdf/pmi_description.urdf (robot description, URDF)
Before this commit: robot pmi_description, 9 links, 8 joints
Links:
- removed link link01
- removed link link02
- removed link link03
- removed link link04
- link base_link: mass 2.1494 -> 2.4727
- link link1: mass 1.2226 -> 1.1285
- link link2: mass 1.2006 -> 1.2748
- link link3: mass 1.0076 -> 1.2621
- link link4: mass 0.85355 -> 0.85956
Joints:
- removed joint q1_act
- removed joint q1_jnt
- removed joint q2_act
- removed joint q2_jnt
- removed joint q3_act
- removed joint q3_jnt
- removed joint q4_act
- removed joint q4_jnt
- added joint jnt1: type revolute, parent base_link, child link1, origin xyz=0 0 0 rpy=3.1416 0 0, axis 0 0 1, limit lower=-100 upper=100 effort=10 velocity=100
- added joint jnt2: type revolute, parent link1, child link2, origin xyz=0 0 -0.22 rpy=1.5708 0 0, axis 0.0063958 0 -0.99998, limit lower=-100 upper=100 effort=10 velocity=100
- added joint jnt3: type revolute, parent link2, child link3, origin xyz=0 -0.23 0 rpy=0 0 -1.5708, axis 0 0 1, limit lower=-100 upper=100 effort=10 velocity=100
- added joint jnt4: type revolute, parent link3, child link4, origin xyz=0.23 0 0 rpy=-3.1416 0 0, axis 0 0 1, limit lower=-100 upper=100 effort=10 velocity=100

Commit message: mujoco vsd applied

File: ros_ws/pmi_description/urdf/pmi_description.urdf (robot description, URDF)
Before this commit: robot pmi_description, 5 links, 4 joints
Links:
- link link1: mass 1.1285 -> 10.0123496865811
- link link2: mass 1.2748 -> 10.4391437674567
- link link3: mass 1.2621 -> 10.3406497234359
- link link4: mass 0.85956 -> 7.01416597186014
Joints:
- joint jnt2: axis 0.0063958 0 -0.99998 -> 0 0 1

Commit message: rl ing...

File: ros_ws/pmi_description/urdf/pmi_description.urdf (robot description, URDF)
Before this commit: robot pmi_description, 5 links, 4 joints
Joints:
- joint jnt2: limit lower=-100 upper=100 effort=10 velocity=100 -> lower=-1.5709 upper=1.5709 effort=10 velocity=100
- joint jnt3: limit lower=-100 upper=100 effort=10 velocity=100 -> lower=-3.1416 upper=3.1416 effort=10 velocity=100
- joint jnt4: limit lower=-100 upper=100 effort=10 velocity=100 -> lower=-1.5709 upper=1.5709 effort=10 velocity=100
