Commit message: PMI 서버/클라이언트 VSD 제어·DXL 통신·IK 경로계획 개선
주요 변경:
- DXL 통신: Indirect Addressing + GroupSyncWrite 도입으로 루프당 트랜잭션 32회 → 4회로 단축;
  USB-CDC 브리지(OpenCM9.04)에서 GroupSyncRead가 -3002 오류를 유발하므로 읽기는
  per-axis readTxRx(22바이트 Indirect Data 블록) 4회로 대체
- VSD 제어: task-space PD + 중력 보상 알고리즘 적용; pmi_vsd_config.txt에서 Ks/Kd/Kt/
  ramp_in_sec 파라미터 로드; trajectory 시작 시 gain ramp-in(0.5 s) 추가로 초기 포화 억제
- 경로계획: kCmdPlanPath 수신 시 현재 encoder 자세로 IK 시작점 anchoring; IK 미수렴
  sample 수 진단 로그 추가
- 로거: ee_cur 계산을 VSD와 동일한 q 소스(j0=motor×gear, j1-3=encoder)로 통일
- 클라이언트 UI: Reset 버튼 추가(하드웨어 오류 초기화), Stop 버튼 → kCmdHoldStop으로 변경
- 프로토콜: kCmdResetError(0x13), kCmdHoldStop(0x14) 추가
- pmi_kinematics 라이브러리 신규 추가(FK, Jacobian, 중력 토크)
- .gitignore: pmi_zero_offsets.txt, analysis/cpp/plots/ 제외 추가

Co-authored-by: Cursor <cursoragent@cursor.com>

File: ros_ws/pmi_description/urdf/pmi_description.urdf (robot description, URDF)
Before this commit: robot pmi_description, 5 links, 4 joints
Joints:
- joint jnt1: limit lower=-100 upper=100 effort=10 velocity=100 -> lower=-3.1416 upper=3.1416 effort=10 velocity=100
- joint jnt3: limit lower=-3.1416 upper=3.1416 effort=10 velocity=100 -> lower=-1.5709 upper=1.5709 effort=10 velocity=100
